File: 02_Electronics/MovuinoShieldPressure/MovuinoShieldPressure.kicad_pcb (KiCad board)
At the start: 2 copper layers, 10 x 34 mm, 3 parts, among them J1 DF12_36NOLEGS_Male, J2 Rext

Commit message: Pressure Shield v1.0
Parts:
- removed J1: DF12_36NOLEGS_Male, Connector_Hirose:Hirose_DF12_DF12C3.0-36DS-0.5V_2x18_P0.50mm_Vertical
- added J3: DF12-36NOLEGS-MALE, MovuinoESP8266:DF12-36-DP-NL, B.Cu at (103.5, 46.5)
- J2: footprint Connector_JST:JST_SH_BM02B-SRSS-TB_1x02-1MP_P1.00mm_Vertical -> Connector_PinHeader_2.54mm:PinHeader_1x02_P2.54mm_Vertical
- R1: value 330 Ohm -> Rref; footprint Resistor_SMD:R_1206_3216Metric -> Resistor_SMD:R_0603_1608Metric_Pad0.98x0.95mm_HandSolder; moved to B.Cu
- moved J2 2.61 mm to (104.0, 35.8), turned to 90 degrees
- moved R1 0.50 mm to (105.0, 56.0), turned to 180 degrees
Connections:
- R1 pad 2: (no net) -> GND
Routing:
- net /ADC: track 0.00 -> 24.0 mm
- net VCC: track 0.00 -> 15.6 mm
- net GND: track 0.00 -> 1.55 mm
Other:
- board size 10 x 34 mm -> 10.5 x 33 mm
- board text added: "ADC"
- board text added: "VCC"

Commit message: update
Parts:
- R1: value Rref -> 330 Ohm
Connections:
- J3 pad 34: Net-(J3-Pad34) -> GND
Routing:
- net GND: track 1.55 -> 2.05 mm

Commit message: design rule ok
Parts:
- added J1: DF12-36NOLEGS-FEMALE, MovuinoESP8266:DF12-36-DP-NL-noPad, F.Cu at (103.5, 46.5)
Routing:
- net GND: track 2.05 -> 5.80 mm, vias 0 -> 1
- net VCC: track 15.6 -> 19.3 mm, vias 0 -> 1
- net /ADC: track 24.0 -> 25.6 mm, vias 0 -> 1
