File: 02_Electronics/MovuinoShieldPressure/MovuinoShieldPressure.kicad_pcb (KiCad board)
At the start: 2 copper layers, 10.5 x 33 mm, 4 parts, among them J1 DF12-36NOLEGS-FEMALE, J2 Rext, J3 DF12-36NOLEGS-MALE

Commit message: update
Other:
- board text added: "Movuino pressure shield v1.0"
- board text added: "designed by Adrien Husson"
- board text removed: "Remplacer trou par empreintes “mounting hole” Changer toutes les dimensions orientation du connecteur 36 nodes Touche espace : reset dx et dy à 0"

Commit message: update for jlcpcb
Parts:
- added REF**: MountingHole_2.1mm, MountingHole:MountingHole_2.1mm, F.Cu at (102.0, 32.0)
- added REF**: MountingHole_2.1mm, MountingHole:MountingHole_2.1mm, F.Cu at (102.0, 61.0)
- renumbered R1 to Rref
Other:
- outline, holes or cut-outs redrawn
- board text added: "Rext"
