File: 02_Electronics/MovuinoShieldPressure/MovuinoShieldPressure.sch (KiCad schematic (older format))
At the start: 3 parts, among them J1 DF12_36NOLEGS_Male, J2 Rext

Commit message: Pressure Shield v1.0
Parts:
- removed J1: DF12_36NOLEGS_Male, Connector_Hirose:Hirose_DF12_DF12C3.0-36DS-0.5V_2x18_P0.50mm_Vertical, symbol Connector_Generic:Conn_02x18_Top_Bottom
- added J3: DF12-36NOLEGS-MALE, MovuinoESP8266:DF12-36-DP-NL, symbol V0.99.3-ESP12-3-mech-eagle-import:DF12-36NOLEGS-MALE
- J2: footprint Connector_JST:JST_EH_S2B-EH_1x02_P2.50mm_Horizontal -> Connector_PinHeader_2.54mm:PinHeader_1x02_P2.54mm_Vertical
- R1: footprint Connector_JST:JST_ACH_BM01B-ACHSS-A-GAN-ETF_1x01-1MP_P1.20mm_Vertical -> Resistor_SMD:R_0603_1608Metric_Pad0.98x0.95mm_HandSolder
Connections:
- net ADC: now also J3.1
- net GND: now also J3.36
- net VCC: now also J3.32
Changed lines of the file:
@@
 F 0 "R1" H 4018 3246 50  0000 L CNN
 F 1 "330 Ohm" H 4018 3155 50  0000 L CNN
-F 2 "Connector_JST:JST_ACH_BM01B-ACHSS-A-GAN-ETF_1x01-1MP_P1.20mm_Vertical" H 3950 3200 50  0001 C CNN
+F 2 "Resistor_SMD:R_0603_1608Metric_Pad0.98x0.95mm_HandSolder" H 3950 3200 50  0001 C CNN
 F 3 "~" H 3950 3200 50  0001 C CNN
 	1    3950 3200
@@
 F 0 "J2" H 4480 2642 50  0000 L CNN
 F 1 "Rext" H 4480 2551 50  0000 L CNN
-F 2 "Connector_JST:JST_EH_S2B-EH_1x02_P2.50mm_Horizontal" H 4400 2650 50  0001 C CNN
+F 2 "Connector_PinHeader_2.54mm:PinHeader_1x02_P2.54mm_Vertical" H 4400 2650 50  0001 C CNN
 F 3 "~" H 4400 2650 50  0001 C CNN
 	1    4400 2650
 	1    0    0    -1
 $EndComp
-Text Label 2400 2150 2    50   ~ 0
-ADC
 Connection ~ 3950 2750
 $Comp
-L power:GND #PWR0103
-U 1 1 614FA73F
-P 2900 3850
-F 0 "#PWR0103" H 2900 3600 50  0001 C CNN
-F 1 "GND" V 2905 3722 50  0000 R CNN
-F 2 "" H 2900 3850 50  0001 C CNN
-F 3 "" H 2900 3850 50  0001 C CNN
-	1    2900 3850
+L V0.99.3-ESP12-3-mech-eagle-import:DF12-36NOLEGS-MALE J3
+U 1 1 615F0003
+P 2650 2900
+F 0 "J3" H 2700 3886 59  0000 C CNN
+F 1 "DF12-36NOLEGS-MALE" H 2700 3781 59  0000 C CNN
+F 2 "MovuinoESP8266:DF12-36-DP-NL" H 2650 2900 50  0001 C CNN
+F 3 "" H 2650 2900 50  0001 C CNN
+	1    2650 2900
+	1    0    0    -1
+$EndComp
+Text Label 2250 2200 2    50   ~ 0
+ADC
+$Comp
+L power:GND #PWR0105
+U 1 1 6162DBE4
+P 3150 3900
+F 0 "#PWR0105" H 3150 3650 50  0001 C CNN
+F 1 "GND" V 3155 3772 50  0000 R CNN
+F 2 "" H 3150 3900 50  0001 C CNN
+F 3 "" H 3150 3900 50  0001 C CNN
+	1    3150 3900
 	0    -1   -1   0
 $EndComp
 $Comp
-L Connector_Generic:Conn_02x18_Top_Bottom J1
-U 1 1 614E8A01
-P 2600 2950
-F 0 "J1" H 2650 3900 50  0000 C CNN
-F 1 "DF12_36NOLEGS_Male" H 2650 1850 50  0000 C CNN
-F 2 "Connector_Hirose:Hirose_DF12_DF12C3.0-36DS-0.5V_2x18_P0.50mm_Vertical" H 2600 2950 50  0001 C CNN
-F 3 "~" H 2600 2950 50  0001 C CNN
-	1    2600 2950
-	1    0    0    -1
-$EndComp
-$Comp
-L power:VCC #PWR0104
-U 1 1 614FB027
-P 2900 3450
-F 0 "#PWR0104" H 2900 3300 50  0001 C CNN
-F 1 "VCC" V 2915 3578 50  0000 L CNN
-F 2 "" H 2900 3450 50  0001 C CNN
-F 3 "" H 2900 3450 50  0001 C CNN
-	1    2900 3450
+L power:VCC #PWR0106
+U 1 1 6162E6D7
+P 3150 3700
+F 0 "#PWR0106" H 3150 3550 50  0001 C CNN
+F 1 "VCC" V 3165 3828 50  0000 L CNN
+F 2 "" H 3150 3700 50  0001 C CNN
+F 3 "" H 3150 3700 50  0001 C CNN
+	1    3150 3700
 	0    1    1    0
 $EndComp

Commit message: update
Connections:
- net GND: now also J3.34
Changed lines of the file:
@@
 	0    1    1    0
 $EndComp
+$Comp
+L power:GND #PWR?
+U 1 1 615F0513
+P 3150 3800
+F 0 "#PWR?" H 3150 3550 50  0001 C CNN
+F 1 "GND" V 3155 3672 50  0000 R CNN
+F 2 "" H 3150 3800 50  0001 C CNN
+F 3 "" H 3150 3800 50  0001 C CNN
+	1    3150 3800
+	0    -1   -1   0
+$EndComp
 $EndSCHEMATC

Commit message: design rule ok
Parts:
- added J1: DF12-36NOLEGS-FEMALE, MovuinoESP8266:DF12-36-DP-NL-noPad, symbol V0.99.3-ESP12-3-mech-eagle-import:DF12-36NOLEGS-FEMALE
Connections:
- net ADC: now also J1.2
- net GND: now also J1.33, J1.35
- net VCC: now also J1.31
Changed lines of the file:
@@
 $EndComp
 $Comp
-L power:GND #PWR?
+L power:GND #PWR0103
 U 1 1 615F0513
 P 3150 3800
-F 0 "#PWR?" H 3150 3550 50  0001 C CNN
+F 0 "#PWR0103" H 3150 3550 50  0001 C CNN
 F 1 "GND" V 3155 3672 50  0000 R CNN
 F 2 "" H 3150 3800 50  0001 C CNN
@@
 	0    -1   -1   0
 $EndComp
+$Comp
+L power:GND #PWR0104
+U 1 1 619F1B45
+P 2250 6200
+F 0 "#PWR0104" H 2250 5950 50  0001 C CNN
+F 1 "GND" V 2255 6072 50  0000 R CNN
+F 2 "" H 2250 6200 50  0001 C CNN
+F 3 "" H 2250 6200 50  0001 C CNN
+	1    2250 6200
+	0    1    1    0
+$EndComp
+$Comp
+L power:VCC #PWR0107
+U 1 1 619F1B4B
+P 2250 6100
+F 0 "#PWR0107" H 2250 5950 50  0001 C CNN
+F 1 "VCC" V 2265 6228 50  0000 L CNN
+F 2 "" H 2250 6100 50  0001 C CNN
+F 3 "" H 2250 6100 50  0001 C CNN
+	1    2250 6100
+	0    -1   -1   0
+$EndComp
+$Comp
+L power:GND #PWR0108
+U 1 1 619F1B51
+P 2250 6300
+F 0 "#PWR0108" H 2250 6050 50  0001 C CNN
+F 1 "GND" V 2255 6172 50  0000 R CNN
+F 2 "" H 2250 6300 50  0001 C CNN
+F 3 "" H 2250 6300 50  0001 C CNN
+	1    2250 6300
+	0    1    1    0
+$EndComp
+$Comp
+L V0.99.3-ESP12-3-mech-eagle-import:DF12-36NOLEGS-FEMALE J1
+U 1 1 61A045A3
+P 2650 5300
+F 0 "J1" H 2700 6286 59  0000 C CNN
+F 1 "DF12-36NOLEGS-FEMALE" H 2700 6181 59  0000 C CNN
+F 2 "MovuinoESP8266:DF12-36-DP-NL-noPad" H 2650 5300 50  0001 C CNN
+F 3 "" H 2650 5300 50  0001 C CNN
+	1    2650 5300
+	1    0    0    -1
+$EndComp
+Text Label 3150 4600 0    50   ~ 0
+ADC
 $EndSCHEMATC
