File: 02_Electronics/SensitivePen_PressureConnector/SensitivePen_PressureConnector.kicad_pcb (KiCad board)
At the start: 2 copper layers, 117.5 x 39.5 mm, 1 part, among them J1 Conn_01x02

Commit message: update (?)
Parts:
- added Ref**: Val**, SensitivePressure:PressurePrint, F.Cu at (180.8, 119.7)
- moved J1 73.9 mm to (179.8, 112.7)
Routing:
- net Net-(J1-Pad2): track 7.25 -> 0.00 mm
- net Net-(J1-Pad1): track 1.01 -> 0.00 mm
- removed copper zone on F.Cu, net Net-(J1-Pad1)
Other:
- outline, holes or cut-outs redrawn

Commit message: design rule ok
Parts:
- removed Ref**: Val**, SensitivePressure:PressurePrint
- added J2: Conn_01x02, SensitivePressure:PressurePrint, F.Cu at (180.8, 119.7)
Other:
- board size 117.5 x 39.5 mm -> 5 x 8.8 mm

Commit message: update
Other:
- outline, holes or cut-outs redrawn
