File: 02_Electronics/shield_v1/shield_v1.kicad_pcb (KiCad board)
At the start: 2 copper layers, 33 x 33 mm, 12 parts, among them J1 Conn_01x02_Male, J2 Conn_01x02_Male, J3 Conn_01x02_Male, J4 DF12_3.0_-36DP-0.5V_86_, J5 DF12_3.0_-36DP-0.5V_86_, J6 FH12-10S-0.5SH(55), U1 FT5316DME

Commit message: update for jlcpcb
Parts:
- added REF**: MountingHole_2.1mm, MountingHole:MountingHole_2.1mm, F.Cu at (52.0, 81.0)
- added REF**: MountingHole_2.1mm, MountingHole:MountingHole_2.1mm, F.Cu at (81.0, 81.0)
- added REF**: MountingHole_2.1mm, MountingHole:MountingHole_2.1mm, F.Cu at (81.0, 52.0)
- added REF**: MountingHole_2.1mm, MountingHole:MountingHole_2.1mm, F.Cu at (52.0, 52.0)
Routing:
- added copper zone on F.Cu, net GND
Other:
- outline, holes or cut-outs redrawn
